File: hardware/18650_Slime/18650_Slime.kicad_pcb (KiCad board)
At the start: 2 copper layers, 59.8 x 32.5 mm, 72 parts, among them J1 IMU_Connector, J10 Conn_01x03_Male, J11 Batt -, J12 Batt -, J2 Conn_01x03_Male, J3 Conn_01x05_Male, J4 Conn_01x05_Male, J5 USB_C_Receptacle_USB2.0, J6 Batt +, J7 Batt +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

Commit message: v0.1.2 of 18650_slime
Parts:
- D1: footprint slimevr_pcb:SOD882 -> 18650_Slime:SOD882
Other:
- board text added: "AUX"
