File: hardware/18650_Slime/18650_Slime.kicad_sch (KiCad schematic)
At the start: 30 parts, among them J1 IMU_Connector, J2 Conn_01x03_Male, J3 Conn_01x05_Male, J4 Conn_01x05_Male, SW1 SW_PWR, U1 BMI160, U2 ESP32-C3-MINI-1, U3 BMM150, U4 M3406, Y1 32.768Hz

Commit message: v0.1.2 of 18650_slime
Parts:
- D1: footprint slimevr_pcb:SOD882 -> 18650_Slime:SOD882
Changed lines of the file:
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@@
   (title_block
     (title "18650_Slime")
-    (date "2022-11-28")
-    (rev "V0.1.0")
+    (date "2022-12-07")
+    (rev "V0.1.3")
     (company "gitlab.com/wigwagwent/18650_slime")
     (comment 1 "Licensed under CERN-OHL-P v2 or later")
@@
       (effects (font (size 1.27 1.27)) (justify left))
     )
-    (property "Footprint" "slimevr_pcb:SOD882" (id 2) (at 16.51 91.44 0)
+    (property "Footprint" "18650_Slime:SOD882" (id 2) (at 16.51 91.44 0)
       (effects (font (size 1.27 1.27)) hide)
     )
@@
     )
     (path "/00000000-0000-0000-0000-000062637b6c"
-      (reference "D1") (unit 1) (value "LESD8D3.3CAT5G") (footprint "slimevr_pcb:SOD882")
+      (reference "D1") (unit 1) (value "LESD8D3.3CAT5G") (footprint "18650_Slime:SOD882")
     )
     (path "/1857a806-cd68-49e5-8da8-50ff7859e548/c8bf2f67-cffd-4d2b-84c8-5d845b70ca23"
