File: hardware/18650_Slime_battery/18650_Slime_battery.kicad_pcb (KiCad board)
At the start: 2 copper layers, 70.5 x 18.2 mm, 37 parts, among them J1 Conn_01x04_Male, Q1 CJ2305, Q2 S8205A, Q3 S8205A, U1 IP2312, U2 FS312F-G

Commit message: V1.0.0 of the battery module done
Parts:
- removed D3: LED, LED_SMD:LED_0603_1608Metric_Pad1.05x0.95mm_HandSolder
- removed R14, R15, R16, R17: 5R, Resistor_SMD:R_0805_2012Metric_Pad1.20x1.40mm_HandSolder
- removed R7: 100R, Resistor_SMD:R_0805_2012Metric_Pad1.20x1.40mm_HandSolder
- added G***: LOGO, 18650_Slime:OpenSourceLogo, F.Cu at (80.6, 65.2)
- B1: footprint 18650:18650_Battery -> 18650_Slime:18650_Battery; moved to B.Cu
- C1, C2, C3, C4, C5, C6, C7, D2, Q1, Q2, Q3, R1, R11, R13, R18, R2, R3, R4, R5, R6, R9, U2: moved to F.Cu
- D1: footprint LED_SMD:LED_0603_1608Metric_Pad1.05x0.95mm_HandSolder -> LED_SMD:LED_0805_2012Metric_Pad1.15x1.40mm_HandSolder; moved to F.Cu
- F1: footprint Capacitor_SMD:C_0805_2012Metric_Pad1.18x1.45mm_HandSolder -> Fuse:Fuse_0805_2012Metric_Pad1.15x1.40mm_HandSolder; moved to F.Cu
- J1: footprint Connector_PinSocket_2.54mm:PinSocket_1x04_P2.54mm_Horizontal -> Connector_PinHeader_2.54mm:PinHeader_1x04_P2.54mm_Horizontal; moved to F.Cu
- L1: footprint 18650:CY54-1.0UH -> 18650_Slime:SMMS0420; moved to F.Cu
- R10: value 30K 1% -> 30K; moved to F.Cu
- R12: value 2R -> 0.5R; moved to F.Cu
- R8: value 120K 1% -> 120K; moved to F.Cu
- U1: footprint 18650:IP2312 -> 18650_Slime:IP2312; moved to F.Cu
- moved D1 64.2 mm to (120.8, 56.5), turned to 0 degrees
- moved R3 63.8 mm to (120.8, 58.5), turned to 180 degrees
- moved R5 60.0 mm to (120.8, 60.5), turned to 180 degrees
- moved R10 53.1 mm to (117.0, 61.0), turned to 90 degrees
- moved C6 52.0 mm to (111.0, 57.3)
- moved C4 51.9 mm to (113.0, 57.3)
- moved R8 50.9 mm to (115.0, 61.0), turned to -90 degrees
- moved F1 50.7 mm to (117.8, 67.8), turned to -90 degrees
- moved C1 47.2 mm to (117.0, 57.3), turned to -90 degrees
- moved R11 45.4 mm to (115.0, 57.3), turned to 90 degrees
- moved D2 43.4 mm to (115.5, 67.3), turned to -90 degrees
- moved Q1 40.6 mm to (108.8, 64.5), turned to 90 degrees
- moved L1 37.3 mm to (107.0, 59.8), turned to 0 degrees
- moved R13 36.5 mm to (59.0, 57.0), turned to 0 degrees
- moved Q2 32.3 mm to (58.5, 67.3)
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Connections:
- J1 pad 1: B_SENSE -> +5V
- J1 pad 3: +5V -> B_SENSE
- Q2 pad 4: Net-(Q2-G1) -> OD
- Q2 pad 5: Net-(Q2-G2) -> OC
- Q3 pad 4: Net-(Q3-G1) -> OD
- Q3 pad 5: Net-(Q3-G2) -> OC
Routing:
- net GND: track 5.21 -> 48.2 mm, vias 21 -> 6
- net -BATT: track 50.1 -> 19.2 mm
- net Net-(U1-D1): track 72.0 -> 41.8 mm
- net B_SENSE: track 46.9 -> 18.5 mm
- net +5P: track 42.2 -> 17.7 mm
- net +5V: track 60.9 -> 36.8 mm, vias 3 -> 0
- net +BATT: track 50.1 -> 71.6 mm, vias 0 -> 2
- net Net-(U1-BAT): track 10.3 -> 28.3 mm
- net Net-(U2-VCC): track 20.0 -> 4.79 mm, vias 2 -> 0
- net OC: track 15.4 -> 23.4 mm
- net Net-(Q2-G1): track 7.80 -> 0.00 mm, vias 2 -> 0
- net Net-(Q3-G1): track 7.28 -> 0.00 mm, vias 2 -> 0
- net Net-(U1-SW): track 7.99 -> 3.33 mm
- net Net-(Q2-D1/D2-Pad1): track 16.0 -> 20.3 mm, vias 0 -> 4
- net Net-(U1-ICHG): track 5.68 -> 2.24 mm
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Other:
- board size 70.5 x 18.2 mm -> 70.5 x 17 mm
- board text added: "${REVISION}"
- board text added: "18650_Slime"
- board text added: "Battery"
- board text added: "For use with SlimeVR Made with <3"
- board text added: "JLCJLCJLCJLC"
- board text added: "License: CERN-OHL-P v2 or later"
- board text added: "gitlab.com/wigwagwent/18650_slime"
- board text removed: "Bottom"

Commit message: V1.0.0 Release, UNTESTED
Parts:
- removed R10: 30K, Resistor_SMD:R_0805_2012Metric_Pad1.20x1.40mm_HandSolder
- removed R8: 120K, Resistor_SMD:R_0805_2012Metric_Pad1.20x1.40mm_HandSolder
- J1: value Conn_01x04_Male -> Conn_01x03_Pin; footprint Connector_PinHeader_2.54mm:PinHeader_1x04_P2.54mm_Horizontal -> Connector_PinHeader_2.54mm:PinHeader_1x03_P2.54mm_Horizontal
Connections:
- J1 pad 3: B_SENSE -> GND
Routing:
- net GND: track 48.2 -> 84.7 mm, vias 6 -> 17
- net B_SENSE: track 18.5 -> 0.00 mm, vias 1 -> 0
- net OC: track 23.4 -> 18.3 mm, vias 2 -> 3
- net OD: track 18.3 -> 17.1 mm, vias 2 -> 3
- net Net-(U1-D1): track 41.8 -> 40.6 mm
Other:
- board text added: "For use with SlimeVR; Made with <3"
- board text added: "GND"
- board text added: "VBUS"
- board text added: "VOUT"
- board text removed: "For use with SlimeVR Made with <3"
