File: hardware/18650_Slime_battery/18650_Slime_battery.kicad_sch (KiCad schematic)
At the start: 38 parts, among them J1 Conn_01x04_Male, Q1 CJ2305, Q2 S8205A, Q3 S8205A, U1 IP2312, U2 FS312F-G

Commit message: V1.0.0 of the battery module done
Parts:
- removed D3: LED, LED_SMD:LED_0603_1608Metric_Pad1.05x0.95mm_HandSolder, symbol Device:LED
- removed R14, R15, R16, R17: 5R, Resistor_SMD:R_0805_2012Metric_Pad1.20x1.40mm_HandSolder, symbol Device:R
- removed R7: 100R, Resistor_SMD:R_0805_2012Metric_Pad1.20x1.40mm_HandSolder, symbol Device:R
- removed TP1: BATT, TestPoint:TestPoint_Pad_D1.0mm, symbol Connector:TestPoint
- B1: footprint 18650:18650_Battery -> 18650_Slime:18650_Battery; symbol 18650:18650_Battery -> 18650_Slime:18650_Battery; LCSC (none) -> DNP
- C1, C2, C4: Extended (none) -> Basic; LCSC (none) -> C45783
- C3, C5: Extended (none) -> Basic; LCSC (none) -> C15850
- C6: Extended (none) -> Basic; LCSC (none) -> C13967
- C7: Extended (none) -> Basic; LCSC (none) -> C49678
- D1: footprint LED_SMD:LED_0603_1608Metric_Pad1.05x0.95mm_HandSolder -> LED_SMD:LED_0805_2012Metric_Pad1.15x1.40mm_HandSolder; Extended (none) -> Basic; LCSC (none) -> C84256
- D2: Extended (none) -> Basic; LCSC (none) -> C8598
- F1: footprint Capacitor_SMD:C_0805_2012Metric_Pad1.18x1.45mm_HandSolder -> Fuse:Fuse_0805_2012Metric_Pad1.15x1.40mm_HandSolder; Extended (none) -> Extended; MANUFACTURER SMD0805B035TF -> (none)
- J1: footprint Connector_PinSocket_2.54mm:PinSocket_1x04_P2.54mm_Horizontal -> Connector_PinHeader_2.54mm:PinHeader_1x04_P2.54mm_Horizontal; LCSC (none) -> DNP
- L1: footprint 18650:CY54-1.0UH -> 18650_Slime:SMMS0420; Extended (none) -> Extended; LCSC (none) -> C133189
- Q1: Extended (none) -> Extended; LCSC (none) -> C8549
- Q2, Q3: symbol 18650:S8205A -> 18650_Slime:S8205A; Extended (none) -> Extended; LCSC (none) -> C436910
- R1: Extended (none) -> Basic; LCSC (none) -> C17436
- R10: value 30K 1% -> 30K; Extended (none) -> Basic; LCSC (none) -> C17621
- R11: Extended (none) -> Extended; LCSC (none) -> C327217
- R12: value 2R -> 0.5R; Extended (none) -> Extended; LCSC (none) -> C327217
- R13, R2, R4: Extended (none) -> Basic; LCSC (none) -> C17513
- R18, R3: Extended (none) -> Basic; LCSC (none) -> C17408
- R5, R9: LCSC (none) -> DNP; now not fitted
- R6: Extended (none) -> Basic; LCSC (none) -> C17737
- R8: value 120K 1% -> 120K; Extended (none) -> Basic; LCSC (none) -> C17436
- U1: footprint 18650:IP2312 -> 18650_Slime:IP2312; symbol 18650:IP2312 -> 18650_Slime:IP2312; Extended (none) -> Extended; LCSC (none) -> C605433
- U2: symbol 18650:FS312F-G -> 18650_Slime:FS312F-G; Extended (none) -> Extended; LCSC (none) -> C82736
Connections:
- net +5V: now also J1.1 (Pin_1); no longer J1.3 (Pin_3)
- net B_SENSE: now also J1.3 (Pin_3); no longer J1.1 (Pin_1)
- net OC: now also Q2.5 (G2), Q3.5 (G2)
- net OD: now also Q2.4 (G1), Q3.4 (G1)
Other:
- note added: "RICHG - R9 135K - 1A 91K - 1.5A 45K - 3A NC - 2.1A"
- note added: "RVSET - R5 NC - 4.2V 43K - 4.3V 75K - 4.35V 100K - 4.4V"
- moved on the sheet: C1

Commit message: V1.0.0 Release, UNTESTED
Parts:
- removed J1: Conn_01x04_Male, Connector_PinHeader_2.54mm:PinHeader_1x04_P2.54mm_Horizontal, symbol Connector:Conn_01x04_Pin
- removed R10: 30K, Resistor_SMD:R_0805_2012Metric_Pad1.20x1.40mm_HandSolder, symbol Device:R_Small
- removed R8: 120K, Resistor_SMD:R_0805_2012Metric_Pad1.20x1.40mm_HandSolder, symbol Device:R_Small
- added J1: Conn_01x03_Pin, Connector_PinHeader_2.54mm:PinHeader_1x03_P2.54mm_Horizontal, symbol Connector:Conn_01x03_Pin
Connections:
- net +5P: now also J1.2 (Pin_2)
- net +5V: now also J1.1 (Pin_1)
- net GND: now also J1.3 (Pin_3)
Other:
- note removed: "Battery Charge Sensor"
- note removed: "Voltage divider by factor of 5"

Commit message: Minor Changes INTESTING
Parts:
- Q2, Q3: value S8205A -> MS8205A; LCSC C436910 -> C5278016 (JLC: C436910)
- U1: LCSC C605433 -> C605432
- U2: value FS312F-G -> DW01C-G; LCSC C82736 -> C35306
Changed lines of the file:
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@@
   (title_block
     (title "18650_Slime_Battery")
-    (date "2023-07-05")
+    (date "2023-07-06")
     (rev "V1.0.0")
     (company "gitlab.com/wigwagwent/18650_slime")
@@
       (effects (font (size 1.27 1.27)))
     )
-    (property "Value" "S8205A" (at 148.59 49.53 0)
+    (property "Value" "MS8205A" (at 148.59 49.53 0)
       (effects (font (size 1.27 1.27)))
     )
@@
       (effects (font (size 1.27 1.27)) hide)
     )
-    (property "Datasheet" "https://datasheet.lcsc.com/lcsc/1912111437_TF-S8205A_C436910.pdf" (at 144.78 52.07 0)
-      (effects (font (size 1.27 1.27)) hide)
-    )
-    (property "LCSC" "C436910" (at 148.59 52.07 0)
+    (property "Datasheet" "https://datasheet.lcsc.com/lcsc/2211211800_MSKSEMI-MS8205A_C5278013.pdf" (at 144.78 52.07 0)
+      (effects (font (size 1.27 1.27)) hide)
+    )
+    (property "LCSC" "C5278016 (JLC: C436910)" (at 148.59 52.07 0)
       (effects (font (size 1.27 1.27)) hide)
     )
@@
       (effects (font (size 1.27 1.27)))
     )
-    (property "Value" "S8205A" (at 148.59 67.31 0)
+    (property "Value" "MS8205A" (at 148.59 67.31 0)
       (effects (font (size 1.27 1.27)))
     )
@@
       (effects (font (size 1.27 1.27)) hide)
     )
-    (property "Datasheet" "https://datasheet.lcsc.com/lcsc/1912111437_TF-S8205A_C436910.pdf" (at 144.78 69.85 0)
-      (effects (font (size 1.27 1.27)) hide)
-    )
-    (property "LCSC" "C436910" (at 148.59 69.85 0)
+    (property "Datasheet" "https://datasheet.lcsc.com/lcsc/2211211800_MSKSEMI-MS8205A_C5278013.pdf" (at 144.78 69.85 0)
+      (effects (font (size 1.27 1.27)) hide)
+    )
+    (property "LCSC" "C5278016 (JLC: C436910)" (at 148.59 69.85 0)
       (effects (font (size 1.27 1.27)) hide)
     )
@@
       (effects (font (size 1.27 1.27)) hide)
     )
-    (property "Datasheet" "https://datasheet.lcsc.com/lcsc/2101081834_INJOINIC-IP2312-4V35_C605433.pdf" (at 50.8 35.56 0)
-      (effects (font (size 1.27 1.27)) hide)
-    )
-    (property "LCSC" "C605433" (at 50.8 35.56 0)
+    (property "Datasheet" "https://datasheet.lcsc.com/lcsc/2009081935_INJOINIC-IP2312U-VSET_C605432.pdf" (at 50.8 35.56 0)
+      (effects (font (size 1.27 1.27)) hide)
+    )
+    (property "LCSC" "C605432" (at 50.8 35.56 0)
       (effects (font (size 1.27 1.27)) hide)
     )
@@
       (effects (font (size 1.27 1.27)))
     )
-    (property "Value" "FS312F-G" (at 150.495 31.75 0)
+    (property "Value" "DW01C-G" (at 150.495 31.75 0)
       (effects (font (size 1.27 1.27)))
     )
@@
       (effects (font (size 1.27 1.27)) hide)
     )
-    (property "LCSC" "C82736" (at 149.86 33.02 0)
-      (effects (font (size 1.27 1.27)) hide)
-    )
+    (property "LCSC" "C35306" (at 149.86 33.02 0)
+      (effects (font (size 1.27 1.27)) hide)
+    )
