File: hardware/18650_Slime_main/18650_Slime_main.kicad_sch (KiCad schematic)
At the start: 55 parts, among them J1 RJ12, J2 USB_C_Receptacle_USB2.0, J3 Conn_01x04_Male, Q1 2N3904, Q2 CJ2305, Q3 2N3904, Q4 CJ2305, SW1 SW_Push, SW2 SW_Push, SW3 SW_Push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

Commit message: V1.0.0 of the battery module done
Parts:
- C1, C2: LCSC (none) -> C28323
- C10: LCSC (none) -> C45783
- C11, C4: LCSC (none) -> C1710
- C3: LCSC (none) -> C49678
- C5, C7, Y1: LCSC (none) -> DNP; now not fitted; now in the parts list
- C6: LCSC (none) -> C1779
- C8: LCSC (none) -> C13967
- C9: LCSC (none) -> C15850
- D1: LCSC (none) -> C5199850
- D2: LCSC (none) -> C2297
- D3: LCSC (none) -> C84256
- D4: LCSC (none) -> C8598
- J1: LCSC (none) -> C3097724
- J2: MANUFACTURER GCT -> (none); MAXIMUM_PACKAGE_HEIGHT 3.31 mm -> (none); PARTREV A3 -> (none); STANDARD Manufacturer Recommendations -> (none)
- J3, U1: LCSC (none) -> DNP
- JP1, TP1, TP2, TP3, TP4, TP5, TP6, TP7: LCSC (none) -> DNP; now left out of the parts list
- L1: LCSC (none) -> C135262
- Q1, Q3: LCSC (none) -> C18536
- Q2, Q4: LCSC (none) -> C8549
- R1, R2, R5: value 4.7K -> 5.1K; LCSC (none) -> C27834
- R10: LCSC C25744 -> C17414
- R11, R12: LCSC (none) -> C27834
- R13, R6: LCSC (none) -> C17429
- R14, R15: LCSC (none) -> C149504
- R16: LCSC (none) -> C17514
- R3: LCSC (none) -> C17414
- R4, R8: LCSC (none) -> C17436
- R7: LCSC (none) -> DNP; now not fitted
- R9: LCSC (none) -> C17593
- U2: LCSC (none) -> C2838502
- U3: LCSC (none) -> C83224
- U4: LCSC (none) -> C558418
Other:
- moved on the sheet: U4

Commit message: V1.0.0 Release, UNTESTED
Parts:
- removed C11: 10nF, Capacitor_SMD:C_0805_2012Metric_Pad1.18x1.45mm_HandSolder, symbol Device:C_Small
- removed D4: B5819W, Diode_SMD:D_SOD-123, symbol Device:D_Schottky
- removed J1: RJ12, 18650:EVERCOM 5501-660211111, symbol Connector:RJ12
- removed J3: Conn_01x04_Male, Connector_PinHeader_2.54mm:PinHeader_1x04_P2.54mm_Horizontal, symbol Connector:Conn_01x04_Pin
- removed Q1, Q3: 2N3904, Package_TO_SOT_SMD:SOT-23-3, symbol Transistor_BJT:2N3904
- removed Q2, Q4: CJ2305, Package_TO_SOT_SMD:SOT-23_Handsoldering, symbol Transistor_FET:DMG2301L
- removed R13: 1K, Resistor_SMD:R_0805_2012Metric_Pad1.20x1.40mm_HandSolder, symbol Device:R_Small
- removed R14, R15: 100K, Resistor_SMD:R_0805_2012Metric_Pad1.20x1.40mm_HandSolder, symbol Device:R_Small
- removed R16: 1M, Resistor_SMD:R_0805_2012Metric_Pad1.20x1.40mm_HandSolder, symbol Device:R_Small
- removed TP3: IO9, TestPoint:TestPoint_Pad_D1.0mm, symbol Connector:TestPoint
- removed TP5: IO2, TestPoint:TestPoint_Pad_D1.0mm, symbol Connector:TestPoint
- removed TP6: GND, TestPoint:TestPoint_Pad_D1.0mm, symbol Connector:TestPoint
- removed TP7: 3v3, TestPoint:TestPoint_Pad_D1.0mm, symbol Connector:TestPoint
- added C11: 1uF, Capacitor_SMD:C_0805_2012Metric_Pad1.18x1.45mm_HandSolder, symbol Device:C
- added C12: 100nF, Capacitor_SMD:C_0805_2012Metric_Pad1.18x1.45mm_HandSolder, symbol Device:C
- added D5: B5819W, Diode_SMD:D_SOD-123, symbol Device:D
- added J1: Conn_01x03_Pin, Connector_PinHeader_2.54mm:PinHeader_1x03_P2.54mm_Horizontal, symbol Connector:Conn_01x03_Pin
- added J2: Conn_01x05_Pin, Connector_PinHeader_2.00mm:PinHeader_1x05_P2.00mm_Vertical, symbol Connector:Conn_01x05_Pin
- added Q1: AO3400A, Package_TO_SOT_SMD:SOT-23, symbol Simulation_SPICE:NMOS
- added Q3: CJ2305, Package_TO_SOT_SMD:SOT-23, symbol Simulation_SPICE:PMOS
- added R13: 10K, Resistor_SMD:R_0805_2012Metric_Pad1.20x1.40mm_HandSolder, symbol Device:R
- added R14, R16: 100K, Resistor_SMD:R_0805_2012Metric_Pad1.20x1.40mm_HandSolder, symbol Device:R
- added R15: 300K, Resistor_SMD:R_0805_2012Metric_Pad1.20x1.40mm_HandSolder, symbol Device:R
- added R17: 1K, Resistor_SMD:R_0805_2012Metric_Pad1.20x1.40mm_HandSolder, symbol Device:R
- added R18: 120K, Resistor_SMD:R_0805_2012Metric_Pad1.20x1.40mm_HandSolder, symbol Device:R_Small
- added R19: 27K, Resistor_SMD:R_0805_2012Metric_Pad1.20x1.40mm_HandSolder, symbol Device:R_Small
- C1, C2: Extended (none) -> Basic; Requirements 16V -> (none)
- C10: value 22uF -> 10uF; Extended (none) -> Basic; LCSC C45783 -> C15850
- C3, C4: Extended (none) -> Basic; Requirements 10V -> (none)
- C5, C7: footprint Capacitor_SMD:C_0805_2012Metric_Pad1.18x1.45mm_HandSolder -> Capacitor_SMD:C_0603_1608Metric; now left out of the parts list
- C6: value 4.7uF -> 10uF; Extended (none) -> Basic; LCSC C1779 -> C15850
- C8, C9, R1, R10, R11, R12, R2, R3, R4: Extended (none) -> Basic
- D1, SW1, SW2, SW3: Extended (none) -> Extended
- D2, D3: footprint LED_SMD:LED_0603_1608Metric_Pad1.05x0.95mm_HandSolder -> Diode_SMD:D_0805_2012Metric_Pad1.15x1.40mm_HandSolder; Extended (none) -> Basic
- J3: renamed from J2; footprint Connector_USB:USB_C_Receptacle_GCT_USB4085 -> Connector_USB:USB_C_Receptacle_XKB_U262-16XN-4BVC11; Extended (none) -> Extended
- L1: footprint Inductor_SMD:L_Wuerth_MAPI-3015 -> 18650:SMMS0420; Extended (none) -> Extended; LCSC C135262 -> C133191
- R5: Extended (none) -> Basic; Requirements 4.7K 1% -> (none)
- R6: Extended (none) -> Basic; Requirements 1K 1% -> (none)
- R7: footprint Resistor_SMD:R_0805_2012Metric_Pad1.20x1.40mm_HandSolder -> Resistor_SMD:R_0603_1608Metric; now left out of the parts list
- R8, R9: Extended (none) -> Basic; Requirements 1% -> (none)
- U1: symbol 18650:BMI160_Module -> 18650_Slime:BMI160_Module
- U2: symbol 18650:ESP32-C3-MINI-1 -> 18650_Slime:ESP32-C3-MINI-1; Extended (none) -> Extended(Standard)
- U3: symbol 18650:M3406 -> 18650_Slime:M3406; Extended (none) -> Extended
- U4: footprint Package_TO_SOT_SMD:SOT-23-6 -> Package_TO_SOT_SMD:SOT-23-6_Handsoldering; Extended (none) -> Extended
- Y1: Requirements 32.768Hz -> (none); now left out of the parts list
Connections:
- net +3V3: now also J2.1 (Pin_1)
- net +5P: now also JP1.1 (A), C12.1, J1.2 (Pin_2), Q3.3 (S), R13.2, R14.2
- net +5V: now also C10.2, Q3.1 (D), R16.2, R18.1
- net GND: now also SW3.1, J1.3 (Pin_3), J2.5 (Pin_5), Q1.3 (S), R19.2; no longer C10.1
- net IO10_SDA: now also J2.2 (Pin_2)
- net IO7_INT2: now also J2.3 (Pin_3)
- net IO8_SCL: now also J2.4 (Pin_4)
- net UNUSED_IO2: now also TP4.1
- net VBUS: now also J3.A4 (VBUS), J3.A9 (VBUS), J3.B4 (VBUS), J3.B9 (VBUS), U4.5 (VP), J1.1 (Pin_1); no longer JP1.1 (A)
- net at SW3.2: now also C11.2, D5.1 (K), R13.1; no longer C10.2
- net B_SENSE renamed IO3_B_SENSE
- net IO3_B_SENSE: now also R18.2, R19.1
- net UNUSED_IO4: no longer names the net of U2.18 (GPIO4/ADC1_CH4)
- net UNUSED_IO4: now also R17.1; no longer TP4.1
- new net: C11.1, C12.2, Q1.1 (D), Q3.2 (G), R14.1
- new net: C10.1, Q1.2 (G), R15.1
- new net IO4_ON/OFF: D5.2 (A), R15.2, R16.1, R17.2
Other:
- note added: "Battery Charge Sensor"
- note added: "Bypass power button for debugging or external switch"
- note added: "Diode D1 is for ESD, don't zap the usb Bitch to solder by hand Leave off if need be"
- note added: "Green LED"
- note added: "R4 prevents ESD"
- note added: "Red LED"
- note added: "Switches are not required for operation. They are usefull for debugging"
- note added: "Voltage divider by a factor of almost 5"
- note removed: "Bypass power button for debugging"
- note removed: "C2: See bootloader docs"
- note removed: "DC/DC Test Point"
- note removed: "Green LED 0603"
- note removed: "R6 prevents ESD"
- note removed: "Red LED 0603"
- moved on the sheet: C1, D2, D3, J3, JP1, R1, R10, R11, R12, R2, R4, R5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

Commit message: Minor Changes INTESTING
Parts:
- removed R4: 120K, Resistor_SMD:R_0805_2012Metric_Pad1.20x1.40mm_HandSolder, symbol Device:R_Small
- D2: LCSC C2297 -> C688883
- R17, R6: LCSC C17429 -> C17513
Connections:
- net GND: now also J3.S1 (SHIELD)
Other:
- note removed: "R4 prevents ESD"
Changed lines of the file:
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@@
   (title_block
     (title "18650_Slime_Main")
-    (date "2023-07-05")
-    (rev "V1.0.0")
+    (date "2023-07-06")
+    (rev "V1.1.0")
     (company "gitlab.com/wigwagwent/18650_slime")
     (comment 1 "Licensed under CERN-OHL-P v2 or later")
@@
   (junction (at 186.69 82.55) (diameter 0) (color 0 0 0 0)
   )
-  (junction (at 129.54 153.67) (diameter 0) (color 0 0 0 0)
+  (junction (at 129.54 151.13) (diameter 0) (color 0 0 0 0)
   )
   (junction (at 154.94 109.22) (diameter 0) (color 0 0 0 0)
@@
     (stroke (width 0) (type default))
   )
-  (wire (pts (xy 130.81 153.67) (xy 129.54 153.67))
+  (wire (pts (xy 130.81 151.13) (xy 129.54 151.13))
     (stroke (width 0) (type default))
   )
@@
     (stroke (width 0) (type default))
   )
-  (wire (pts (xy 121.92 153.67) (xy 121.92 152.4))
-    (stroke (width 0) (type default))
-  )
   (polyline (pts (xy 200.66 13.97) (xy 234.95 13.97))
     (stroke (width 0) (type default))
@@
     (stroke (width 0) (type default))
   )
-  (wire (pts (xy 129.54 147.32) (xy 129.54 153.67))
-    (stroke (width 0) (type default))
-  )
   (wire (pts (xy 40.64 180.34) (xy 39.37 180.34))
     (stroke (width 0) (type default))
@@
     (stroke (width 0) (type default))
   )
-  (wire (pts (xy 121.92 153.67) (xy 129.54 153.67))
+  (wire (pts (xy 121.92 151.13) (xy 129.54 151.13))
     (stroke (width 0) (type default))
   )
@@
     (stroke (width 0) (type default))
   )
+  (wire (pts (xy 121.92 147.32) (xy 121.92 151.13))
+    (stroke (width 0) (type default))
+  )
   (polyline (pts (xy 66.04 156.21) (xy 66.04 199.39))
     (stroke (width 0) (type default))
@@
     (stroke (width 0) (type default))
   )
+  (wire (pts (xy 129.54 147.32) (xy 129.54 151.13))
+    (stroke (width 0) (type default))
+  )
   (polyline (pts (xy 71.12 157.48) (xy 71.12 180.34))
     (stroke (width 0) (type default))
@@
     (effects (font (size 1.27 1.27) (thickness 0.254) bold) (justify left bottom))
   )
-  (text "R4 prevents ESD" (at 116.84 157.48 0)
-    (effects (font (size 0.75 0.75)) (justify left bottom))
-  )
   (global_label "IO7_INT2" (shape output) (at 40.64 180.34 0) (fields_autoplaced)
     (effects (font (size 1.27 1.27)) (justify left))
@@
       (effects (font (size 1.27 1.27)) hide)
     )
-    (property "LCSC" "C2297" (at 242.57 130.81 0)
+    (property "LCSC" "C688883" (at 242.57 130.81 0)
       (effects (font (size 1.27 1.27)) hide)
     )
@@
       (effects (font (size 1.27 1.27)) hide)
     )
-    (property "LCSC" "C17429" (at 231.14 107.95 0)
+    (property "LCSC" "C17513" (at 231.14 107.95 0)
       (effects (font (size 1.27 1.27)) hide)
     )
@@
     )
   )
-  (symbol (lib_id "Device:R_Small") (at 121.92 149.86 0) (unit 1)
-    (in_bom yes) (on_board yes) (dnp no)
-    (property "Reference" "R4" (at 123.19 148.59 0)
-      (effects (font (size 1.27 1.27)) (justify left))
-    )
-    (property "Value" "120K" (at 123.19 151.13 0)
-      (effects (font (size 1.27 1.27)) (justify left))
-    )
-    (property "Footprint" "Resistor_SMD:R_0805_2012Metric_Pad1.20x1.40mm_HandSolder" (at 121.92 149.86 0)
-      (effects (font (size 1.27 1.27)) hide)
-    )
-    (property "Datasheet" "~" (at 121.92 149.86 0)
-      (effects (font (size 1.27 1.27)) hide)
-    )
-    (property "LCSC" "C17436" (at 121.92 149.86 0)
-      (effects (font (size 1.27 1.27)) hide)
-    )
-    (property "Extended" "Basic" (at 121.92 149.86 0)
-      (effects (font (size 1.27 1.27)) hide)
-    )
-    (pin "1")
-    (pin "2")
-    (instances
-      (project "18650_Slime_main"
-        (path "/196a8dd5-5fd6-4c7f-ae4a-0104bd82e61b"
-          (reference "R4") (unit 1)
-        )
-      )
-    )
-  )
   (symbol (lib_id "Device:C_Small") (at 129.54 30.48 0) (unit 1)
     (in_bom yes) (on_board yes) (dnp no)
@@
     )
   )
-  (symbol (lib_id "power:GND") (at 130.81 153.67 90) (unit 1)
+  (symbol (lib_id "power:GND") (at 130.81 151.13 90) (unit 1)
     (in_bom yes) (on_board yes) (dnp no)
-    (property "Reference" "#PWR018" (at 137.16 153.67 0)
+    (property "Reference" "#PWR018" (at 137.16 151.13 0)
       (effects (font (size 1.27 1.27)) hide)
     )
-    (property "Value" "GND" (at 135.89 153.67 90)
+    (property "Value" "GND" (at 135.89 151.13 90)
       (effects (font (size 1.27 1.27)))
     )
-    (property "Footprint" "" (at 130.81 153.67 0)
+    (property "Footprint" "" (at 130.81 151.13 0)
       (effects (font (size 1.27 1.27)) hide)
     )
-    (property "Datasheet" "" (at 130.81 153.67 0)
+    (property "Datasheet" "" (at 130.81 151.13 0)
       (effects (font (size 1.27 1.27)) hide)
     )
@@
       (effects (font (size 1.27 1.27)) hide)
     )
-    (property "LCSC" "C17429" (at 34.29 49.53 0)
+    (property "LCSC" "C17513" (at 34.29 49.53 0)
       (effects (font (size 1.27 1.27)) hide)
     )
